Commit message: catkinized package

File: robots/uplift_description.URDF (robot description, URDF)
Before this commit: robot uplift_description, 5 links, 4 joints
Joints:
- joint arm: limit lower=-1.3 upper=1.2 effort=10 velocity=0.5 -> lower=-1.3 upper=1.4 effort=10 velocity=0.5

Commit message: moved camera to right side and decreased spine limit

File: robots/uplift_description.URDF (robot description, URDF)
Before this commit: robot uplift_description, 5 links, 4 joints
Joints:
- joint camera: origin xyz=-0.32184 -0.25391 -0.02305 rpy=-3.1339 5.3352E-18 1.5708 -> xyz=-0.135 -0.18 -0.02305 rpy=-3.1339 5.3352E-18 1.5708
- joint spine: limit lower=0 upper=0.4 effort=10 velocity=0.02 -> lower=0 upper=0.27 effort=10 velocity=0.02

Commit message: limit adjusted

File: robots/uplift_description.URDF (robot description, URDF)
Before this commit: robot uplift_description, 5 links, 4 joints
Joints:
- joint arm: limit lower=-1.3 upper=1.4 effort=10 velocity=0.5 -> lower=-1.4 upper=1.2 effort=10 velocity=0.5
